File: Sensor-HAT.kicad_sch (KiCad schematic)
At the start: 112 parts, among them J1 RPi GPIO 2x20, J2 1-Wire GND/DQ/3V3, J3 UART (e.g. PMS5003), J4 PM sensor (SEN6x/SEN5x), J5 Qwiic / STEMMA QT, J6 GPIO expansion (DNP), J7 XIAO D0-D6, J8 XIAO 5V-D7, Q1 AO3401A, Q2 AO3400A, Q3 AO3400A, SW1 Button, U1 SCD41-D-R2, U12 74LV1T125, U13 SGP41, U14 LM66100, U15 LM66100, U2 SHT40, U3 ICS-43434, U4 CAT24C32, U5 AP2112K-3.3, U6 AP2112K-3.3, U7 VEML7700-TT, U8 SRV05-4, U9 AP2112K-3.3

Commit message: Tidy up the schematic: no overlapping texts (no electrical change)
- gen_sch.py places reference/value beside the body, above/below or above
  the top-right corner, depending on where the pins leave, so they no longer
  cross wires and labels; PWR_FLAG labels get a short stub
- design.py: XIAO series resistors R33-R43 in one row, crowded parts moved
  apart, long header texts split into two lines
- patch_lib.py hides pin names that the EasyEDA symbols draw over their
  graphics and removes the pin-1 dots
- schematic PDF re-exported

Netlist identical (74 nets, 112 parts), ERC 0, DRC 0 with schematic parity.

Co-Authored-By: Claude Opus 5.5 <noreply@anthropic.com>
Other:
- note added: "(LDOs on while Pi 3V3 or XIAO 3V3 is present)"
- note added: "J3 pin 1 = 3.3 V (JP1) or switched/fused 5 V (JP3), never both"
- note added: "Power: Pi 5 V or XIAO USB 5 V via ideal diodes -> +5V -> AP2112K-3.3 LDOs"
- note added: "UART (GPIO14/15 / XIAO D6/D7) + GPIO17: series R, ESD"
- note removed: "Power: Pi 5 V or XIAO USB 5 V via ideal diodes -> +5V -> AP2112K-3.3 LDOs, enabled by Pi 3V3 OR XIAO 3V3"
- note removed: "UART (GPIO14/15 / XIAO D6/D7) + GPIO17: series R, ESD, J3 pin 1 = 3.3 V (JP1) or switched/fused 5 V (JP3), never both"
- moved on the sheet: C12, C20, C24, C26, C29, C30, C31, F1, J6, R16, R22, R23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
